Commit message: fixing launch file

File: src/urdf_description/urdf/URDF.xacro (robot description, xacro)
@@ -1,7 +1,7 @@
 <?xml version="1.0" ?>
 <robot name="URDF" xmlns:xacro="http://www.ros.org/wiki/xacro">
-<xacro:include filename="$(find URDF_description)/urdf/materials.xacro" />
-<xacro:include filename="$(find URDF_description)/urdf/URDF.trans" />
-<xacro:include filename="$(find URDF_description)/urdf/URDF.gazebo" />
+<xacro:include filename="$(find urdf_description)/urdf/materials.xacro" />
+<xacro:include filename="$(find urdf_description)/urdf/URDF.trans" />
+<xacro:include filename="$(find urdf_description)/urdf/URDF.gazebo" />
 <link name="base_link">
   <inertial>
@@ -13,5 +13,5 @@
     <origin xyz="0 0 0" rpy="0 0 0"/>
     <geometry>
-      <mesh filename="file://$(find URDF_description)/meshes/base_link.stl" scale="0.001 0.001 0.001"/>
+      <mesh filename="file://$(find urdf_description)/meshes/base_link.stl" scale="0.001 0.001 0.001"/>
     </geometry>
     <material name="silver"/>
@@ -20,5 +20,5 @@
     <origin xyz="0 0 0" rpy="0 0 0"/>
     <geometry>
-      <mesh filename="file://$(find URDF_description)/meshes/base_link.stl" scale="0.001 0.001 0.001"/>
+      <mesh filename="file://$(find urdf_description)/meshes/base_link.stl" scale="0.001 0.001 0.001"/>
     </geometry>
   </collision>
@@ -33,5 +33,5 @@
     <origin xyz="-0.254 0.2915 -0.4537" rpy="0 0 0"/>
     <geometry>
-      <mesh filename="file://$(find URDF_description)/meshes/pushrod_left_1.stl" scale="0.001 0.001 0.001"/>
+      <mesh filename="file://$(find urdf_description)/meshes/pushrod_left_1.stl" scale="0.001 0.001 0.001"/>
     </geometry>
     <material name="silver"/>
@@ -40,5 +40,5 @@
     <origin xyz="-0.254 0.2915 -0.4537" rpy="0 0 0"/>
     <geometry>
-      <mesh filename="file://$(find URDF_description)/meshes/pushrod_left_1.stl" scale="0.001 0.001 0.001"/>
+      <mesh filename="file://$(find urdf_description)/meshes/pushrod_left_1.stl" scale="0.001 0.001 0.001"/>
     </geometry>
   </collision>
@@ -53,5 +53,5 @@
     <origin xyz="-0.0 0.355 -0.4791" rpy="0 0 0"/>
     <geometry>
-      <mesh filename="file://$(find URDF_description)/meshes/diff_bar_1.stl" scale="0.001 0.001 0.001"/>
+      <mesh filename="file://$(find urdf_description)/meshes/diff_bar_1.stl" scale="0.001 0.001 0.001"/>
     </geometry>
     <material name="silver"/>
@@ -60,5 +60,5 @@
     <origin xyz="-0.0 0.355 -0.4791" rpy="0 0 0"/>
     <geometry>
-      <mesh filename="file://$(find URDF_description)/meshes/diff_bar_1.stl" scale="0.001 0.001 0.001"/>
+      <mesh filename="file://$(find urdf_description)/meshes/diff_bar_1.stl" scale="0.001 0.001 0.001"/>
     </geometry>
   </collision>
@@ -73,5 +73,5 @@
     <origin xyz="0.254 0.2915 -0.4537" rpy="0 0 0"/>
     <geometry>
-      <mesh filename="file://$(find URDF_description)/meshes/pushrod_right_1.stl" scale="0.001 0.001 0.001"/>
+      <mesh filename="file://$(find urdf_description)/meshes/pushrod_right_1.stl" scale="0.001 0.001 0.001"/>
     </geometry>
     <material name="silver"/>
@@ -80,5 +80,5 @@
     <origin xyz="0.254 0.2915 -0.4537" rpy="0 0 0"/>
     <geometry>
-      <mesh filename="file://$(find URDF_description)/meshes/pushrod_right_1.stl" scale="0.001 0.001 0.001"/>
+      <mesh filename="file://$(find urdf_description)/meshes/pushrod_right_1.stl" scale="0.001 0.001 0.001"/>
     </geometry>
   </collision>
@@ -93,5 +93,5 @@
     <origin xyz="0.28213 -0.0 -0.2931" rpy="0 0 0"/>
     <geometry>
-      <mesh filename="file://$(find URDF_description)/meshes/bracket_right_1.stl" scale="0.001 0.001 0.001"/>
+      <mesh filename="file://$(find urdf_description)/meshes/bracket_right_1.stl" scale="0.001 0.001 0.001"/>
     </geometry>
     <material name="silver"/>
@@ -100,5 +100,5 @@
     <origin xyz="0.28213 -0.0 -0.2931" rpy="0 0 0"/>
     <geometry>
-      <mesh filename="file://$(find URDF_description)/meshes/bracket_right_1.stl" scale="0.001 0.001 0.001"/>
+      <mesh filename="file://$(find urdf_description)/meshes/bracket_right_1.stl" scale="0.001 0.001 0.001"/>
     </geometry>
   </collision>
@@ -113,5 +113,5 @@
     <origin xyz="-0.28213 -0.0 -0.2931" rpy="0 0 0"/>
     <geometry>
-      <mesh filename="file://$(find URDF_description)/meshes/bracket_left_1.stl" scale="0.001 0.001 0.001"/>
+      <mesh filename="file://$(find urdf_description)/meshes/bracket_left_1.stl" scale="0.001 0.001 0.001"/>
     </geometry>
     <material name="silver"/>
@@ -120,5 +120,5 @@
     <origin xyz="-0.28213 -0.0 -0.2931" rpy="0 0 0"/>
     <geometry>
-      <mesh filename="file://$(find URDF_description)/meshes/bracket_left_1.stl" scale="0.001 0.001 0.001"/>
+      <mesh filename="file://$(find urdf_description)/meshes/bracket_left_1.stl" scale="0.001 0.001 0.001"/>
     </geometry>
   </collision>
@@ -133,5 +133,5 @@
     <origin xyz="0.70223 -0.26313 -0.3312" rpy="0 0 0"/>
     <geometry>
-      <mesh filename="file://$(find URDF_description)/meshes/pushrod_right_1.stl" scale="0.001 0.001 0.001"/>
+      <mesh filename="file://$(find urdf_description)/meshes/pushrod_right_1.stl" scale="0.001 0.001 0.001"/>
     </geometry>
     <material name="silver"/>
@@ -140,5 +140,5 @@
     <origin xyz="0.70223 -0.26313 -0.3312" rpy="0 0 0"/>
     <geometry>
-      <mesh filename="file://$(find URDF_description)/meshes/pushrod_right_1.stl" scale="0.001 0.001 0.001"/>
+      <mesh filename="file://$(find urdf_description)/meshes/pushrod_right_1.stl" scale="0.001 0.001 0.001"/>
     </geometry>
   </collision>
@@ -153,5 +153,5 @@
     <origin xyz="0.18877 0.26313 -0.3312" rpy="0 0 0"/>
     <geometry>
-      <mesh filename="file://$(find URDF_description)/meshes/pushrod_left_1.stl" scale="0.001 0.001 0.001"/>
+      <mesh filename="file://$(find urdf_description)/meshes/pushrod_left_1.stl" scale="0.001 0.001 0.001"/>
     </geometry>
     <material name="silver"/>
@@ -160,5 +160,5 @@
     <origin xyz="0.18877 0.26313 -0.3312" rpy="0 0 0"/>
     <geometry>
-      <mesh filename="file://$(find URDF_description)/meshes/pushrod_left_1.stl" scale="0.001 0.001 0.001"/>
+      <mesh filename="file://$(find urdf_description)/meshes/pushrod_left_1.stl" scale="0.001 0.001 0.001"/>
     </geometry>
   </collision>
@@ -173,5 +173,5 @@
     <origin xyz="-0.30753 0.22225 -0.2931" rpy="0 0 0"/>
     <geometry>
-      <mesh filename="file://$(find URDF_description)/meshes/rocker_left_1.stl" scale="0.001 0.001 0.001"/>
+      <mesh filename="file://$(find urdf_description)/meshes/rocker_left_1.stl" scale="0.001 0.001 0.001"/>
     </geometry>
     <material name="silver"/>
@@ -180,5 +180,5 @@
     <origin xyz="-0.30753 0.22225 -0.2931" rpy="0 0 0"/>
     <geometry>
-      <mesh filename="file://$(find URDF_description)/meshes/rocker_left_1.stl" scale="0.001 0.001 0.001"/>
+      <mesh filename="file://$(find urdf_description)/meshes/rocker_left_1.stl" scale="0.001 0.001 0.001"/>
     </geometry>
   </collision>
@@ -193,5 +193,5 @@
     <origin xyz="0.30753 0.22225 -0.2931" rpy="0 0 0"/>
     <geometry>
-      <mesh filename="file://$(find URDF_description)/meshes/rocker_right_1.stl" scale="0.001 0.001 0.001"/>
+      <mesh filename="file://$(find urdf_description)/meshes/rocker_right_1.stl" scale="0.001 0.001 0.001"/>
     </geometry>
     <material name="silver"/>
@@ -200,5 +200,5 @@
     <origin xyz="0.30753 0.22225 -0.2931" rpy="0 0 0"/>
     <geometry>
-      <mesh filename="file://$(find URDF_description)/meshes/rocker_right_1.stl" scale="0.001 0.001 0.001"/>
+      <mesh filename="file://$(find urdf_description)/meshes/rocker_right_1.stl" scale="0.001 0.001 0.001"/>
     </geometry>
   </collision>
@@ -213,5 +213,5 @@
     <origin xyz="-0.23933 0.40457 -0.03727" rpy="0 0 0"/>
     <geometry>
-      <mesh filename="file://$(find URDF_description)/meshes/motor_left_front_1.stl" scale="0.001 0.001 0.001"/>
+      <mesh filename="file://$(find urdf_description)/meshes/motor_left_front_1.stl" scale="0.001 0.001 0.001"/>
     </geometry>
     <material name="silver"/>
@@ -220,5 +220,5 @@
     <origin xyz="-0.23933 0.40457 -0.03727" rpy="0 0 0"/>
     <geometry>
-      <mesh filename="file://$(find URDF_description)/meshes/motor_left_front_1.stl" scale="0.001 0.001 0.001"/>
+      <mesh filename="file://$(find urdf_description)/meshes/motor_left_front_1.stl" scale="0.001 0.001 0.001"/>
     </geometry>
   </collision>
@@ -233,5 +233,5 @@
     <origin xyz="-0.24083 0.381 -0.0137" rpy="0 0 0"/>
     <geometry>
-      <mesh filename="file://$(find URDF_description)/meshes/coupling_left_front_1.stl" scale="0.001 0.001 0.001"/>
+      <mesh filename="file://$(find urdf_description)/meshes/coupling_left_front_1.stl" scale="0.001 0.001 0.001"/>
     </geometry>
     <material name="silver"/>
@@ -240,5 +240,5 @@
     <origin xyz="-0.24083 0.381 -0.0137" rpy="0 0 0"/>
     <geometry>
-      <mesh filename="file://$(find URDF_description)/meshes/coupling_left_front_1.stl" scale="0.001 0.001 0.001"/>
+      <mesh filename="file://$(find urdf_description)/meshes/coupling_left_front_1.stl" scale="0.001 0.001 0.001"/>
     </geometry>
   </collision>
@@ -253,5 +253,5 @@
     <origin xyz="-0.23933 -0.35743 -0.03727" rpy="0 0 0"/>
     <geometry>
-      <mesh filename="file://$(find URDF_description)/meshes/motor_left_rear_1.stl" scale="0.001 0.001 0.001"/>
+      <mesh filename="file://$(find urdf_description)/meshes/motor_left_rear_1.stl" scale="0.001 0.001 0.001"/>
     </geometry>
     <material name="silver"/>
@@ -260,5 +260,5 @@
     <origin xyz="-0.23933 -0.35743 -0.03727" rpy="0 0 0"/>
     <geometry>
-      <mesh filename="file://$(find URDF_description)/meshes/motor_left_rear_1.stl" scale="0.001 0.001 0.001"/>
+      <mesh filename="file://$(find urdf_description)/meshes/motor_left_rear_1.stl" scale="0.001 0.001 0.001"/>
     </geometry>
   </collision>
@@ -273,5 +273,5 @@
     <origin xyz="0.23933 0.35743 -0.03727" rpy="0 0 0"/>
     <geometry>
-      <mesh filename="file://$(find URDF_description)/meshes/motor_right_front_1.stl" scale="0.001 0.001 0.001"/>
+      <mesh filename="file://$(find urdf_description)/meshes/motor_right_front_1.stl" scale="0.001 0.001 0.001"/>
     </geometry>
     <material name="silver"/>
@@ -280,5 +280,5 @@
     <origin xyz="0.23933 0.35743 -0.03727" rpy="0 0 0"/>
     <geometry>
-      <mesh filename="file://$(find URDF_description)/meshes/motor_right_front_1.stl" scale="0.001 0.001 0.001"/>
+      <mesh filename="file://$(find urdf_description)/meshes/motor_right_front_1.stl" scale="0.001 0.001 0.001"/>
     </geometry>
   </collision>
@@ -293,5 +293,5 @@
     <origin xyz="0.23933 -0.35743 -0.03727" rpy="0 0 0"/>
     <geometry>
-      <mesh filename="file://$(find URDF_description)/meshes/motor_right_rear_1.stl" scale="0.001 0.001 0.001"/>
+      <mesh filename="file://$(find urdf_description)/meshes/motor_right_rear_1.stl" scale="0.001 0.001 0.001"/>
     </geometry>
     <material name="silver"/>
@@ -300,5 +300,5 @@
     <origin xyz="0.23933 -0.35743 -0.03727" rpy="0 0 0"/>
     <geometry>
-      <mesh filename="file://$(find URDF_description)/meshes/motor_right_rear_1.stl" scale="0.001 0.001 0.001"/>
+      <mesh filename="file://$(find urdf_description)/meshes/motor_right_rear_1.stl" scale="0.001 0.001 0.001"/>
     </geometry>
   </collision>
@@ -313,5 +313,5 @@
     <origin xyz="-0.24203 -0.381 -0.0137" rpy="0 0 0"/>
     <geometry>
-      <mesh filename="file://$(find URDF_description)/meshes/coupling_left_rear_1.stl" scale="0.001 0.001 0.001"/>
+      <mesh filename="file://$(find urdf_description)/meshes/coupling_left_rear_1.stl" scale="0.001 0.001 0.001"/>
     </geometry>
     <material name="silver"/>
@@ -320,5 +320,5 @@
     <origin xyz="-0.24203 -0.381 -0.0137" rpy="0 0 0"/>
     <geometry>
-      <mesh filename="file://$(find URDF_description)/meshes/coupling_left_rear_1.stl" scale="0.001 0.001 0.001"/>
+      <mesh filename="file://$(find urdf_description)/meshes/coupling_left_rear_1.stl" scale="0.001 0.001 0.001"/>
     </geometry>
   </collision>
@@ -333,5 +333,5 @@
     <origin xyz="0.24083 -0.381 -0.0137" rpy="0 0 0"/>
     <geometry>
-      <mesh filename="file://$(find URDF_description)/meshes/coupling_right_rear_1.stl" scale="0.001 0.001 0.001"/>
+      <mesh filename="file://$(find urdf_description)/meshes/coupling_right_rear_1.stl" scale="0.001 0.001 0.001"/>
     </geometry>
     <material name="silver"/>
@@ -340,5 +340,5 @@
     <origin xyz="0.24083 -0.381 -0.0137" rpy="0 0 0"/>
     <geometry>
-      <mesh filename="file://$(find URDF_description)/meshes/coupling_right_rear_1.stl" scale="0.001 0.001 0.001"/>
+      <mesh filename="file://$(find urdf_description)/meshes/coupling_right_rear_1.stl" scale="0.001 0.001 0.001"/>
     </geometry>
   </collision>
@@ -353,5 +353,5 @@
     <origin xyz="0.24083 0.381 -0.0137" rpy="0 0 0"/>
     <geometry>
-      <mesh filename="file://$(find URDF_description)/meshes/coupling_right_front_1.stl" scale="0.001 0.001 0.001"/>
+      <mesh filename="file://$(find urdf_description)/meshes/coupling_right_front_1.stl" scale="0.001 0.001 0.001"/>
     </geometry>
     <material name="silver"/>
@@ -360,5 +360,5 @@
     <origin xyz="0.24083 0.381 -0.0137" rpy="0 0 0"/>
     <geometry>
-      <mesh filename="file://$(find URDF_description)/meshes/coupling_right_front_1.stl" scale="0.001 0.001 0.001"/>
+      <mesh filename="file://$(find urdf_description)/meshes/coupling_right_front_1.stl" scale="0.001 0.001 0.001"/>
     </geometry>
   </collision>
@@ -373,5 +373,5 @@
     <origin xyz="-0.31883 0.381158 -0.013819" rpy="0 0 0"/>
     <geometry>
-      <mesh filename="file://$(find URDF_description)/meshes/wheel_left_front_1.stl" scale="0.001 0.001 0.001"/>
+      <mesh filename="file://$(find urdf_description)/meshes/wheel_left_front_1.stl" scale="0.001 0.001 0.001"/>
     </geometry>
     <material name="silver"/>
@@ -380,5 +380,5 @@
     <origin xyz="-0.31883 0.381158 -0.013819" rpy="0 0 0"/>
     <geometry>
-      <mesh filename="file://$(find URDF_description)/meshes/wheel_left_front_1.stl" scale="0.001 0.001 0.001"/>
+      <mesh filename="file://$(find urdf_description)/meshes/wheel_left_front_1.stl" scale="0.001 0.001 0.001"/>
     </geometry>
   </collision>
@@ -393,5 +393,5 @@
     <origin xyz="-0.32003 -0.381158 -0.013819" rpy="0 0 0"/>
     <geometry>
-      <mesh filename="file://$(find URDF_description)/meshes/wheel_left_rear_1.stl" scale="0.001 0.001 0.001"/>
+      <mesh filename="file://$(find urdf_description)/meshes/wheel_left_rear_1.stl" scale="0.001 0.001 0.001"/>
     </geometry>
     <material name="silver"/>
@@ -400,5 +400,5 @@
     <origin xyz="-0.32003 -0.381158 -0.013819" rpy="0 0 0"/>
     <geometry>
-      <mesh filename="file://$(find URDF_description)/meshes/wheel_left_rear_1.stl" scale="0.001 0.001 0.001"/>
+      <mesh filename="file://$(find urdf_description)/meshes/wheel_left_rear_1.stl" scale="0.001 0.001 0.001"/>
     </geometry>
   </collision>
@@ -413,5 +413,5 @@
     <origin xyz="0.31883 -0.381158 -0.013819" rpy="0 0 0"/>
     <geometry>
-      <mesh filename="file://$(find URDF_description)/meshes/wheel_right_rear_1.stl" scale="0.001 0.001 0.001"/>
+      <mesh filename="file://$(find urdf_description)/meshes/wheel_right_rear_1.stl" scale="0.001 0.001 0.001"/>
     </geometry>
     <material name="silver"/>
@@ -420,5 +420,5 @@
     <origin xyz="0.31883 -0.381158 -0.013819" rpy="0 0 0"/>
     <geometry>
-      <mesh filename="file://$(find URDF_description)/meshes/wheel_right_rear_1.stl" scale="0.001 0.001 0.001"/>
+      <mesh filename="file://$(find urdf_description)/meshes/wheel_right_rear_1.stl" scale="0.001 0.001 0.001"/>
     </geometry>
   </collision>
@@ -433,5 +433,5 @@
     <origin xyz="0.31883 0.381158 -0.013819" rpy="0 0 0"/>
     <geometry>
-      <mesh filename="file://$(find URDF_description)/meshes/wheel_right_front_1.stl" scale="0.001 0.001 0.001"/>
+      <mesh filename="file://$(find urdf_description)/meshes/wheel_right_front_1.stl" scale="0.001 0.001 0.001"/>
     </geometry>
     <material name="silver"/>
@@ -440,5 +440,5 @@
     <origin xyz="0.31883 0.381158 -0.013819" rpy="0 0 0"/>
     <geometry>
-      <mesh filename="file://$(find URDF_description)/meshes/wheel_right_front_1.stl" scale="0.001 0.001 0.001"/>
+      <mesh filename="file://$(find urdf_description)/meshes/wheel_right_front_1.stl" scale="0.001 0.001 0.001"/>
     </geometry>
   </collision>
@@ -453,5 +453,5 @@
     <origin xyz="-0.160015 0.293904 -0.5241" rpy="0 0 0"/>
     <geometry>
-      <mesh filename="file://$(find URDF_description)/meshes/hull_mid_1.stl" scale="0.001 0.001 0.001"/>
+      <mesh filename="file://$(find urdf_description)/meshes/hull_mid_1.stl" scale="0.001 0.001 0.001"/>
     </geometry>
     <material name="silver"/>
@@ -460,5 +460,5 @@
     <origin xyz="-0.160015 0.293904 -0.5241" rpy="0 0 0"/>
     <geometry>
-      <mesh filename="file://$(find URDF_description)/meshes/hull_mid_1.stl" scale="0.001 0.001 0.001"/>
+      <mesh filename="file://$(find urdf_description)/meshes/hull_mid_1.stl" scale="0.001 0.001 0.001"/>
     </geometry>
   </collision>
@@ -473,5 +473,5 @@
     <origin xyz="-0.3 -0.0 -0.6991" rpy="0 0 0"/>
     <geometry>
-      <mesh filename="file://$(find URDF_description)/meshes/hull_top_1.stl" scale="0.001 0.001 0.001"/>
+      <mesh filename="file://$(find urdf_description)/meshes/hull_top_1.stl" scale="0.001 0.001 0.001"/>
     </geometry>
     <material name="silver"/>
@@ -480,10 +480,8 @@
     <origin xyz="-0.3 -0.0 -0.6991" rpy="0 0 0"/>
     <geometry>
-      <mesh filename="file://$(find URDF_description)/meshes/hull_top_1.stl" scale="0.001 0.001 0.001"/>
-    </geometry>
-  </collision>
-</link>
-<<<<<<< HEAD
-=======
+      <mesh filename="file://$(find urdf_description)/meshes/hull_top_1.stl" scale="0.001 0.001 0.001"/>
+    </geometry>
+  </collision>
+</link>
 <link name="lidar_link">
   <inertial>
@@ -508,5 +506,4 @@
   </collision>
 </link>
->>>>>>> faa0e8358101bead9ad2591501b71885c5b5ade5
 <joint name="left_pushbar_joint" type="fixed">
   <origin xyz="-0.18877 0.09187 -0.1479" rpy="0 0 0"/>
@@ -544,99 +541,55 @@
   <child link="pushrod_left_rocker_1"/>
 </joint>
-<<<<<<< HEAD
-<joint name="left_rocker_to_bracket (1)" type="fixed">
-=======
 <joint name="left_rocker_to_bracket" type="fixed">
->>>>>>> faa0e8358101bead9ad2591501b71885c5b5ade5
   <origin xyz="0.0254 -0.22225 0.0" rpy="0 0 0"/>
   <parent link="bracket_left_1"/>
   <child link="rocker_left_1"/>
 </joint>
-<<<<<<< HEAD
-<joint name="right_rocker_to_bracket (1)" type="fixed">
-=======
 <joint name="right_rocker_to_bracket" type="fixed">
->>>>>>> faa0e8358101bead9ad2591501b71885c5b5ade5
   <origin xyz="-0.0254 -0.22225 0.0" rpy="0 0 0"/>
   <parent link="bracket_right_1"/>
   <child link="rocker_right_1"/>
 </joint>
-<<<<<<< HEAD
-<joint name="lf_motor_to_rocker (1)" type="fixed">
-=======
 <joint name="lf_motor_to_rocker" type="fixed">
->>>>>>> faa0e8358101bead9ad2591501b71885c5b5ade5
   <origin xyz="-0.0682 -0.18232 -0.25583" rpy="0 0 0"/>
   <parent link="rocker_left_1"/>
   <child link="motor_left_front_1"/>
 </joint>
-<<<<<<< HEAD
-<joint name="lf_coupling_to_motor (1)" type="fixed">
-=======
 <joint name="lf_coupling_to_motor" type="fixed">
->>>>>>> faa0e8358101bead9ad2591501b71885c5b5ade5
   <origin xyz="0.0015 0.02357 -0.02357" rpy="0 0 0"/>
   <parent link="motor_left_front_1"/>
   <child link="coupling_left_front_1"/>
 </joint>
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